File: electrical/press_electrical_prudentia_v1.0/OSCHSSP_electrical_design_prudentia_v1.0.kicad_sch (KiCad schematic)
At the start: 21 parts, among them J1 Mains 120V 60Hz 15Amax, J2 LCD-I2C, SW1 SW_DIP_x01, SW2 RotaryEncoder_Switch, U1 34.81-9024, U1 MAX31855, U2 34.81-9024

Commit message: updated elec
Parts:
- added J3: Conn_01x06, symbol Connector_Generic:Conn_01x06
Connections:
- net +5V: now also J3.1 (Pin_1)
- net GND: now also J3.2 (Pin_2)
- net SSR1: now also A1.20 (A1); no longer A1.14 (D11)
- net SSR2: now also A1.19 (A0); no longer A1.15 (D12)
- net SD_MOSI: now reaches A1.12 (D9)
- net SD_MOSI: now also J3.3 (Pin_3)
- net SD_SS: now reaches A1.13 (D10)
- net SD_SS: now also J3.4 (Pin_4)
- new net SD_MISO: A1.15 (D12), J3.6 (Pin_6)
- new net SD_SCK: A1.14 (D11), J3.5 (Pin_5)
