File: electrical/Nano_KiCAD-master/NanoV3.3.kicad_sch (KiCad schematic)
At the start: 32 parts, among them IC1 FT232RL, IC2 LM1117IMPX-5.0, IC3 328P-MUR, J1 Conn_1x15, J2 Conn_1x15, J3 Conn_Mini_USB, J4 Conn_2x3, SW1 RESET, Y1 16MHz

Commit message: v2 of elec separating gui and improved part selection
Parts:
- renumbered C2 to C25, C9 to C26, C1 to C3, C7 to C4, C3 to C6, C8 to C7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
