File: electrical/Nano_KiCAD-master/NanoV3.3.kicad_sch (KiCad schematic)
At the start: 32 parts, among them IC11 328P-MUR, IC12 FT232RL, IC3 LM1117IMPX-5.0, J11 Conn_Mini_USB, J2 Conn_1x15, J3 Conn_1x15, J4 Conn_2x3, SW4 RESET, Y1 16MHz

Commit message: local push
Parts:
- renumbered C8 to C10, C9 to C11, C25 to C12, C26 to C13, C3 to C5, C4 to C6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
